Commit message: nucobot -> lisa

File: src/lisa_simulator/lisa_description/lisa/urdf/kinect_camera.urdf.xacro (robot description, xacro)
@@ -13,5 +13,5 @@
           <origin xyz="0 0 0" rpy="0 0 0" />
           <geometry>
-            <mesh filename="package://nucobot_description/lisa/meshes/kinect_camera_simple.dae"/>
+            <mesh filename="package://lisa_description/lisa/meshes/kinect_camera_simple.dae"/>
           </geometry>
         </visual>
@@ -19,5 +19,5 @@
           <origin xyz="0 0 0" rpy="0 0 0" />
           <geometry>
-            <mesh filename="package://nucobot_description/lisa/meshes/kinect_camera_simple.dae"/>
+            <mesh filename="package://lisa_description/lisa/meshes/kinect_camera_simple.dae"/>
           </geometry>
         </collision>

File: src/lisa_simulator/lisa_description/lisa/urdf/lisa.urdf.xacro (robot description, xacro)
@@ -1,5 +1,5 @@
 <?xml version="1.0"?>
 <robot name="lisa" xmlns:xacro="http://www.ros.org/wiki/xacro">
-  <xacro:include filename="$(find nucobot_description)/lisa/urdf/materials.xacro" />
+  <xacro:include filename="$(find lisa_description)/lisa/urdf/materials.xacro" />
   <property name="M_PI" value="3.1415926535897931" />
   <link name="base_footprint"/>
@@ -200,10 +200,10 @@
   </gazebo>
   <!-- Kinect -->
-  <xacro:include filename="$(find nucobot_description)/lisa/urdf/kinect_camera.urdf.xacro" />
+  <xacro:include filename="$(find lisa_description)/lisa/urdf/kinect_camera.urdf.xacro" />
   <xacro:kinect_camera name="kinect" parent="base_link">
     <origin xyz="${0.178/2} 0 ${0.3/2}" rpy="0.0 0.0 0.0"/>
   </xacro:kinect_camera>
   <!-- Generic camera
-  <xacro:include filename="$(find nucobot_description)/lisa/urdf/generic_camera.urdf.xacro" />
+  <xacro:include filename="$(find lisa_description)/lisa/urdf/generic_camera.urdf.xacro" />
   <xacro:generic_camera name="generic_camera" parent="base_link" ros_topic="/sensors/generic_camera/image" cam_info_topic="/sensors/generic_camera/camera_info" update_rate="15" res_x="320" res_y="240" image_format="L8" hfov="75">
     <origin xyz="${base_x_size/2-camera_link/2} 0 ${base_z_size/2 + camera_link/2}" rpy="0 0 3.14"/>
